Commit message: Add YOLO+Claude detection pipeline, CLIP visual DB, and multi-medicine scan
- detect_all_medicines(): YOLO handles Thai meds locally, Claude handles English/unknown,
  results merged with no duplicates — YOLO tells Claude which positions to skip
- YOLOv8n trained on 150 real images + 12 labeled mixed-basket scenes (5 Thai med classes)
- CLIP embedding DB (ViT-B-32) as secondary identifier for low-confidence Thai items
- auto_label.py: auto-generates YOLO bbox labels from single-medicine images using
  yellow basket background masking
- thai_visual.py: CLIP collect/build_db/match workflow
- /scan command: captures basket, detects all medicines, presents markdown table
- image_pub.py: fake_result returns NG to keep TMflow Vision1 loop running
- URDF: table Y offset -0.14m, suction_link visual-only (no collision)
- New STL meshes: basket, table, suction_tool, environment

Co-Authored-By: Claude Sonnet 4.6 <noreply@anthropic.com>

File: tmr_ros2/tm_description/xacro/macro.tm5-900-nominal.urdf.xacro (robot description, xacro)
@@ -274,5 +274,39 @@
     <origin rpy="0.000000 0.000000 0.000000" xyz="0.000000 0.000000 0.000000" />
   </joint>
+  <!-- Suction tool attached at flange — visual only, no collision to avoid false self-collision in MoveIt2 -->
+  <link name="${prefix}suction_link">
+    <visual>
+      <origin rpy="0 0 0" xyz="0 0 0"/>
+      <geometry>
+        <mesh filename="package://tm_description/meshes/tm5-900/visual/suction_tool.stl" scale="1 1 1"/>
+      </geometry>
+      <material name="dark_grey">
+        <color rgba="0.3 0.3 0.3 1.0"/>
+      </material>
+    </visual>
+  </link>
+  <joint name="${prefix}suction_fixed_joint" type="fixed">
+    <parent link="${prefix}flange"/>
+    <child link="${prefix}suction_link"/>
+    <origin rpy="0 0 0" xyz="0 0 0"/>
+  </joint>
 <!--LinkDescription-->
+  <!-- Static environment: table, basket, bins from TableWArm.fbx -->
+  <link name="environment_link">
+    <visual>
+      <origin rpy="0 0 0" xyz="0 0 0"/>
+      <geometry>
+        <mesh filename="package://tm_description/meshes/tm5-900/visual/environment.stl" scale="0.8 0.8 0.8"/>
+      </geometry>
+      <material name="light_grey">
+        <color rgba="0.8 0.8 0.8 1.0"/>
+      </material>
+    </visual>
+  </link>
+  <joint name="environment_fixed_joint" type="fixed">
+    <parent link="${prefix}base"/>
+    <child link="environment_link"/>
+    <origin rpy="0 0 3.14159" xyz="0 -0.14 -0.9073"/>
+  </joint>
   </xacro:macro>
 </robot>
