Commit message: Add scaled FBX environment mesh to RViz, increase pick/place speed, return home after placing
- Export table+basket trays from FBX at 0.79 scale (corrects FBX 1.26x oversizing) and add as visual-only env_scene link
- Remove old conflicting environment_link from tm5x macro
- Speed up pick/place travel moves (0.2->0.5, 0.05->0.1, 0.15->0.4)
- Return arm to home pose after placing in bin so vision loop has consistent scan position

File: tmr_ros2/tm5-900_moveit_config/config/tm5-900.urdf.xacro (robot description, xacro)
@@ -7,3 +7,24 @@
     <xacro:include filename="tm5-900.ros2_control.xacro" />
     <xacro:tm5-900_ros2_control name="FakeSystem" initial_positions_file="$(arg initial_positions_file)"/>
+    <!-- Visual-only environment reference: table + 4 basket trays from FBX,
+         scaled 0.79x to match real robot dimensions (FBX was ~1.26x oversized,
+         confirmed by comparing arm_1/arm_2 link lengths to URDF DH params) -->
+    <link name="env_scene">
+        <visual>
+            <origin xyz="0 0 0" rpy="0 0 0"/>
+            <geometry>
+                <mesh filename="package://tm_description/meshes/environment/env_scene.stl" scale="1 1 1"/>
+            </geometry>
+            <material name="env_table_material">
+                <color rgba="0.7 0.7 0.7 1.0"/>
+            </material>
+        </visual>
+    </link>
+    <!-- Mesh was exported in FBX-world coords scaled by 0.79, so shift by
+         -0.79 * robot-base empty origin (0,0,0.784) = (0,0,-0.61936) -->
+    <joint name="env_scene_joint" type="fixed">
+        <parent link="link_0"/>
+        <child link="env_scene"/>
+        <origin xyz="0 0 -0.61936" rpy="0 0 0"/>
+    </joint>
 </robot>

File: tmr_ros2/tm_description/xacro/macro.tm5-900-nominal.urdf.xacro (robot description, xacro)
@@ -291,22 +291,4 @@
     <origin rpy="0 0 0" xyz="0 0 0"/>
   </joint>
-<!--LinkDescription-->
-  <!-- Static environment: table, basket, bins from TableWArm.fbx -->
-  <link name="environment_link">
-    <visual>
-      <origin rpy="0 0 0" xyz="0 0 0"/>
-      <geometry>
-        <mesh filename="package://tm_description/meshes/tm5-900/visual/environment.stl" scale="0.8 0.8 0.8"/>
-      </geometry>
-      <material name="light_grey">
-        <color rgba="0.8 0.8 0.8 1.0"/>
-      </material>
-    </visual>
-  </link>
-  <joint name="environment_fixed_joint" type="fixed">
-    <parent link="${prefix}base"/>
-    <child link="environment_link"/>
-    <origin rpy="0 0 3.14159" xyz="0 -0.14 -0.9073"/>
-  </joint>
   </xacro:macro>
 </robot>

File: tmr_ros2/tm_description/xacro/macro.tm5x-900-nominal.urdf.xacro (robot description, xacro)
@@ -274,4 +274,27 @@
     <origin rpy="0.000000 0.000000 0.000000" xyz="0.000000 0.000000 0.000000" />
   </joint>
+  <!-- Suction tool attached at flange -->
+  <link name="${prefix}suction_link">
+    <visual>
+      <origin rpy="0 0 0" xyz="0 0 0"/>
+      <geometry>
+        <mesh filename="package://tm_description/meshes/tm5-900/visual/suction_tool.stl" scale="1 1 1"/>
+      </geometry>
+      <material name="dark_grey">
+        <color rgba="0.3 0.3 0.3 1.0"/>
+      </material>
+    </visual>
+    <collision>
+      <origin rpy="0 0 0" xyz="0 0 0"/>
+      <geometry>
+        <mesh filename="package://tm_description/meshes/tm5-900/collision/suction_tool_c.stl" scale="1 1 1"/>
+      </geometry>
+    </collision>
+  </link>
+  <joint name="${prefix}suction_fixed_joint" type="fixed">
+    <parent link="${prefix}flange"/>
+    <child link="${prefix}suction_link"/>
+    <origin rpy="0 0 0" xyz="0 0 0"/>
+  </joint>
 <!--LinkDescription-->
   </xacro:macro>
